Commit message: Added inertial components

File: description/robot_core.xacro (robot description, xacro)
@@ -37,4 +37,7 @@
             </geometry>
         </collision>
+        <xacro:inertial_box mass="2" x="0.4" y="0.25" z="0.11">
+            <origin xyz="0.2 0 0.05" rpy="0 0 0"/>
+        </xacro:inertial_box>
     </link>
     <!-- LEFT WHEEL LINK -->
@@ -57,4 +60,7 @@
             </geometry>
         </collision>
+        <xacro:inertial_cylinder mass="0.1" length="0.02" radius="0.067">
+            <origin xyz="0 0 0" rpy="0 0 0"/>
+        </xacro:inertial_cylinder>
     </link>
     <!-- RIGHT WHEEL LINK -->
@@ -77,4 +83,7 @@
             </geometry>
         </collision>
+        <xacro:inertial_cylinder mass="0.1" length="0.02" radius="0.067">
+            <origin xyz="0 0 0" rpy="0 0 0"/>
+        </xacro:inertial_cylinder>
     </link>
     <!-- CASTOR WHEEL LINK-->
@@ -96,4 +105,7 @@
             </geometry>
         </collision>
+        <xacro:inertial_sphere mass="0.01" adius="0.001">
+            <origin xyz="0 0 0" rpy="0 0 0"/>
+        </xacro:inertial_sphere>
     </link>
 </robot>
