Commit message: Ros2 control added

File: description/lidar.xacro (robot description, xacro)
@@ -4,5 +4,5 @@
         <parent link="chassis"/>
         <child link="laser_frame"/>
-        <origin xyz="0.1 0 0.130" rpy="0 0 0"/>
+        <origin xyz="0.3 0 0.14" rpy="0 0 0"/>
     </joint>
     <link name="laser_frame">

File: description/robot.urdf.xacro (robot description, xacro)
@@ -1,6 +1,12 @@
 <?xml version="1.0"?>
 <robot xmlns:xacro="http://www.ros.org/wiki/xacro"  name="robot">
+    <xacro:arg name="use_ros2_control" default="true"/>
     <xacro:include filename="robot_core.xacro" />
-    <xacro:include filename="gazebo_control.xacro" />
+    <xacro:if value="$(arg use_ros2_control)">
+        <xacro:include filename="ros2_control.xacro" />
+    </xacro:if>
+    <xacro:unless value="$(arg use_ros2_control)">
+        <xacro:include filename="gazebo_control.xacro" />
+    </xacro:unless>
     <xacro:include filename="lidar.xacro" />
 </robot>

File: description/robot_core.xacro (robot description, xacro)
@@ -103,10 +103,10 @@
         <parent link="chassis"/>
         <child link="caster_wheel"/>
-        <origin xyz="0.390 0 -0.01"/>
+        <origin xyz="0.390 0 -0.015"/>
     </joint>
     <link name="caster_wheel">
         <visual>
             <geometry>
-                <sphere radius="0.01"/>
+                <sphere radius="0.02"/>
             </geometry>
             <material name='black'/>
@@ -114,8 +114,8 @@
         <collision>
             <geometry>
-                <sphere radius="0.01"/>
+                <sphere radius="0.02"/>
             </geometry>
         </collision>
-        <xacro:inertial_sphere mass="0.01" radius="0.001">
+        <xacro:inertial_sphere mass="0.01" radius="0.02">
             <origin xyz="0 0 0" rpy="0 0 0"/>
         </xacro:inertial_sphere>
